File: Schematic/SchematGrupowy.kicad_sch (KiCad schematic)
At the start: 64 parts, among them J1 USB_C_Receptacle_USB2.0_14P, J2 UART1, J3 UART2, J4 Micro_SD_Card_Det1, J5 LCD, J6 Conn_Coaxial, J7 Programing1, J8 Programing2, SW1 SW_Wuerth_450301014042, SW2 RotaryEncoder_Switch_MP, U1 STM32F411CEUx, U2 BMI160, U3 NEO-M8N, U4 TP4056-42-ESOP8, U5 MCP1700-3302E, U6 STM32F303K8Tx

Commit message: Resolve DRC issues and pour ground planes
Parts:
- BT1: footprint Battery:BatteryHolder_MPD_BK-18650-PC2 -> Connector_JST:JST_PH_S2B-PH-K_1x02_P2.00mm_Horizontal
Changed lines of the file:
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@@
 			)
 		)
-		(property "Footprint" "Battery:BatteryHolder_MPD_BK-18650-PC2"
+		(property "Footprint" "Connector_JST:JST_PH_S2B-PH-K_1x02_P2.00mm_Horizontal"
 			(at 204.47 244.856 90)
 			(effects
